Commit message: wip

File: client/f10_racecar/racecar_differential.urdf (robot description, URDF)
Before this commit: robot racecar, 21 links, 20 joints
Links:
- link left_front_wheel: geometry collision cylinder length=0.045 radius=0.05; visual mesh filename=meshes/left_front_wheel.dae
- link left_rear_wheel: geometry collision cylinder length=0.045 radius=0.05; visual mesh filename=meshes/left_rear_wheel.dae
- link right_front_wheel: geometry collision cylinder length=0.045 radius=0.05; visual mesh filename=meshes/right_front_wheel.dae
- link right_rear_wheel: geometry collision cylinder length=0.045 radius=0.05; visual mesh filename=meshes/right_rear_wheel.dae

Commit message: wip

File: client/f10_racecar/racecar_differential.urdf (robot description, URDF)
Before this commit: robot racecar, 21 links, 20 joints
Joints:
- removed joint diff2_ring_chassis
- removed joint diff2_sideA_ring
- removed joint diff2_sideB_ring
- removed joint diff2_spiderA_ring
- removed joint diff2_spiderB_ring
- removed joint diff_ring_chassis
- removed joint diff_sideA_ring
- removed joint diff_sideB_ring
- removed joint diff_spiderA_ring
- removed joint diff_spiderB_ring
- removed joint hokuyo_joint
- removed joint left_front_wheel_joint
- removed joint left_rear_wheel_joint
- removed joint left_steering_hinge_joint
- removed joint right_front_wheel_joint
- removed joint right_rear_wheel_joint
- removed joint right_steering_hinge_joint
- removed joint zed_camera_joint
- removed joint zed_camera_left_joint
- removed joint zed_camera_right_joint
- added joint diff2RingChassis: type continuous, parent chassis, child diff2_ring, origin xyz=0.32 0.0 0.0 rpy=0 0 0, axis 0 1 0
- added joint diff2SideARing: type continuous, parent diff2_ring, child diff2_sideA, origin xyz=0.0 0.0 0.0 rpy=0 0 0, axis 0 1 0
- added joint diff2SideBRing: type continuous, parent diff2_ring, child diff2_sideB, origin xyz=0.0 0.0 0.0 rpy=0 0 0, axis 0 1 0
- added joint diff2SpiderARing: type continuous, parent diff2_ring, child diff2_spiderA, origin xyz=0.0 0.0 0.0 rpy=0 0 1.570795, axis 0 1 0
- added joint diff2SpiderBRing: type continuous, parent diff2_ring, child diff2_spiderB, origin xyz=0.0 0.0 0.0 rpy=0 0 -1.570795, axis 0 1 0
- added joint diffRingChassis: type continuous, parent chassis, child diff_ring, origin xyz=0.0 0.0 0. rpy=0 0 0, axis 0 1 0
- added joint diffSideARing: type continuous, parent diff_ring, child diff_sideA, origin xyz=0.0 0.0 0.0 rpy=0 0 0, axis 0 1 0
- added joint diffSideBRing: type continuous, parent diff_ring, child diff_sideB, origin xyz=0.0 0.0 0.0 rpy=0 0 0, axis 0 1 0
- added joint diffSpiderARing: type continuous, parent diff_ring, child diff_spiderA, origin xyz=0.0 0.0 0.0 rpy=0 0 1.570795, axis 0 1 0
- added joint diffSpiderBRing: type continuous, parent diff_ring, child diff_spiderB, origin xyz=0.0 0.0 0.0 rpy=0 0 -1.570795, axis 0 1 0
- added joint hokuyoJoint: type fixed, parent chassis, child laser, origin xyz=0.265 0.0 0.075 rpy=0 0 0, axis 0 0 1
- added joint leftFrontWheelJoint: type continuous, parent left_steering_hinge, child left_front_wheel, origin xyz=0 0 0 rpy=1.5708 0 0, axis 0 0 -1, limit effort=10 velocity=100
- added joint leftRearWheelJoint: type fixed, parent diff_sideA, child left_rear_wheel, origin xyz=0 0.1 0 rpy=1.5708 0 0
- added joint leftSteeringHingeJoint: type revolute, parent chassis, child left_steering_hinge, origin xyz=0.325 0.1 0 rpy=0 1.5708 0, axis -1 0 0, limit lower=-1.0 upper=1.0 effort=10 velocity=100
- added joint rightFrontWheelJoint: type continuous, parent right_steering_hinge, child right_front_wheel, origin xyz=0 0 0 rpy=1.5708 0 0, axis 0 0 -1, limit effort=10 velocity=100
- added joint rightRearWheelJoint: type fixed, parent diff_sideB, child right_rear_wheel, origin xyz=0 -0.1 0 rpy=1.5708 0 0
- added joint rightSteeringHingeJoint: type continuous, parent chassis, child right_steering_hinge, origin xyz=0.325 -0.1 0 rpy=0 1.5708 0, axis -1 0 0, limit lower=-1.0 upper=1.0 effort=10 velocity=100
- added joint zedCameraJoint: type fixed, parent chassis, child zed_camera_link, origin xyz=0.390 0 0.04 rpy=0 0 0, axis 0 0 1
- added joint zedCameraLeftJoint: type fixed, parent zed_camera_link, child camera_link, origin xyz=0 0.06 0 rpy=0 0 0, axis 0 0 1
- added joint zedCameraRightJoint: type fixed, parent zed_camera_link, child zed_camera_right_link, origin xyz=0 -0.06 0 rpy=0 0 0, axis 0 0 1
